Commit message: Update model with material of Al and chnage the unit of inertial moment

File: models/sample.urdf (robot description, URDF)
Before this commit: robot sample_robot, 10 links, 9 joints
Links:
- link bracket_1_link: mass 1.702 -> 0.609588
- link bracket_2_link: mass 4.758 -> 1.703374
- link bracket_3_link: mass 3.912 -> 1.400547
- link bracket_4_link: mass 3.912 -> 1.400547
- link bracket_5_link: mass 4.097 -> 1.466917
- link bracket_6_link: mass 2.888 -> 1.033966
- link bracket_7_link: mass 0.825 -> 0.29527
- link end_effector_link: mass 0.733 -> 0.26231
